File: samples/av-connector-breakout/av-connector-breakout.kicad_pcb (KiCad board)
At the start: 2 copper layers, 39.7 x 29.5 mm, 12 parts

Commit message: clean up repo
Parts:
- TP10, TP11, TP7, TP8, TP9: moved to B.Cu
- moved TP11 22.5 mm to (170.2, 73.8), turned to 180 degrees
- moved TP10 22.1 mm to (168.0, 73.8), turned to 180 degrees
- moved TP9 21.7 mm to (165.8, 73.8), turned to 180 degrees
- moved TP8 21.3 mm to (163.5, 73.8), turned to 180 degrees
- moved TP7 21.0 mm to (161.2, 73.8), turned to 180 degrees
- moved TP6 7.29 mm to (172.5, 73.8)
- moved TP5 7.10 mm to (170.2, 73.8)
- moved TP4 6.76 mm to (168.0, 73.8)
- moved TP3 6.43 mm to (165.8, 73.8)
- moved TP2 6.25 mm to (163.5, 73.8)
- moved TP1 5.98 mm to (161.2, 73.8)
Routing:
- net /PSP_BLUE_LUME_PB: track 39.2 -> 14.8 mm, vias 1 -> 0
- net /PSP_WAKE: track 37.7 -> 13.4 mm, vias 1 -> 0
- net /PSP_VIDEO_DETECT: track 35.9 -> 12.2 mm, vias 1 -> 0
- net /PSP_UART_VCC: track 34.3 -> 10.8 mm, vias 1 -> 0
- net /PSPRX: track 32.3 -> 10.2 mm, vias 1 -> 0
- net /GND: track 29.0 -> 20.7 mm
- net /RED_LUMA_PR: track 22.5 -> 14.6 mm
- net /LUMA_Y: track 20.1 -> 13.4 mm
- net /UART_GND: track 18.5 -> 12.1 mm
- net /PSPTX: track 16.8 -> 10.8 mm
- net /PSPMICIN: track 15.0 -> 10.2 mm
Other:
- board size 39.7 x 29.5 mm -> 14 x 16.6 mm
- board text added: "1"
- board text added: "11"
- board text added: "12"
- board text added: "2"
- board text added: "3"
- board text added: "4"
- board text added: "5"
- board text added: "6"
- board text added: "7"
- board text added: "8"
- board text added: "9"
- board text removed: "LUMA_Y"
- board text removed: "Mic input"
- board text removed: "PSP RX"
- board text removed: "PSP TX"
- board text removed: "PSP WAKE"
- board text removed: "PSP_BLUE_LUME_PB"
- board text removed: "RED_LUMA_PR"
- board text removed: "UART GND"
- board text removed: "UART VCC"
- board text removed: "VIDEO DETECT"
- board text removed: "VIDEO GND"
